File: motors.kicad_sch (KiCad schematic)
At the start: 0 parts

Commit message: Ostensibly finish power sheet
Parts:
- added C17, C24, C26, C28: 100u, Capacitor_SMD:C_1206_3216Metric, symbol Device:C
- added C18, C23, C25, C27: 100n, Capacitor_SMD:C_0603_1608Metric, symbol Device:C
- added D1, D6, D7, D8: 1N5819WS, Diode_SMD:D_SOD-323, symbol Diode:1N5819WS
- added Q1, Q2, Q3, Q4: NMOS, Package_TO_SOT_SMD:SOT-23, symbol Simulation_SPICE:NMOS
- added R12, R15, R16, R17: 10k, Resistor_SMD:R_0603_1608Metric, symbol Device:R
- added TP1: MOT1P, TestPoint:TestPoint_Pad_2.0x2.0mm, symbol Connector:TestPoint
- added TP2: MOT1M, TestPoint:TestPoint_Pad_2.0x2.0mm, symbol Connector:TestPoint
- added TP3: MOT2P, TestPoint:TestPoint_Pad_2.0x2.0mm, symbol Connector:TestPoint
- added TP4: MOT2M, TestPoint:TestPoint_Pad_2.0x2.0mm, symbol Connector:TestPoint
- added TP5: MOT3P, TestPoint:TestPoint_Pad_2.0x2.0mm, symbol Connector:TestPoint
- added TP6: MOT3M, TestPoint:TestPoint_Pad_2.0x2.0mm, symbol Connector:TestPoint
- added TP7: MOT4P, TestPoint:TestPoint_Pad_2.0x2.0mm, symbol Connector:TestPoint
- added TP8: MOT4M, TestPoint:TestPoint_Pad_2.0x2.0mm, symbol Connector:TestPoint
Connections:
- new net: D1.2 (A), Q1.1 (D), TP2.1
- new net: D7.2 (A), Q3.1 (D), TP6.1
- new net: D6.2 (A), Q2.1 (D), TP4.1
- new net: D8.2 (A), Q4.1 (D), TP8.1
- new net +BATT: C17.1, C18.1, C23.1, C24.1, C25.1, C26.1, C27.1, C28.1, D1.1 (K), D6.1 (K), D7.1 (K), D8.1 (K), TP1.1, TP3.1, TP5.1, TP7.1
- new net GND: C17.2, C18.2, C23.2, C24.2, C25.2, C26.2, C27.2, C28.2, Q1.3 (S), Q2.3 (S), Q3.3 (S), Q4.3 (S), R12.2, R15.2, R16.2, R17.2
- new net MOT1: Q1.2 (G), R12.1
- new net MOT2: Q2.2 (G), R15.1
- new net MOT3: Q3.2 (G), R16.1
- new net MOT4: Q4.2 (G), R17.1
Other:
- note added: "MOTOR DRIVE"

Commit message: Random changes
Parts:
- added U16: DRV8328ARUYR, easyeda2kicad:WQFN-28_L4.0-W4.0-P0.40-TL-EP2.6, symbol easyeda2kicad:DRV8328ARUYR
Changed lines of the file:
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@@
 		(dnp no)
 		(property "Reference" "C17"
-			(at 44.196 35.814 0)
+			(at 43.688 35.814 0)
 			(show_name no)
 			(do_not_autoplace no)
@@
 		)
 		(property "Value" "100u"
-			(at 43.942 37.846 0)
+			(at 43.434 37.846 0)
 			(show_name no)
 			(do_not_autoplace no)
@@
 	)
 	(symbol
+		(lib_id "easyeda2kicad:DRV8328ARUYR")
+		(at 44.45 140.97 0)
+		(unit 1)
+		(body_style 1)
+		(exclude_from_sim no)
+		(in_bom yes)
+		(on_board yes)
+		(in_pos_files yes)
+		(dnp no)
+		(fields_autoplaced yes)
+		(property "Reference" "U16"
+			(at 44.45 163.83 0)
+			(show_name no)
+			(do_not_autoplace no)
+			(effects
+				(font
+					(size 1.27 1.27)
+				)
+			)
+		)
+		(property "Value" "DRV8328ARUYR"
+			(at 44.45 166.37 0)
+			(show_name no)
+			(do_not_autoplace no)
+			(effects
+				(font
+					(size 1.27 1.27)
+				)
+			)
+		)
+		(property "Footprint" "easyeda2kicad:WQFN-28_L4.0-W4.0-P0.40-TL-EP2.6"
+			(at 44.45 166.37 0)
+			(hide yes)
+			(show_name no)
+			(do_not_autoplace no)
+			(effects
+				(font
+					(size 1.27 1.27)
+				)
+			)
+		)
+		(property "Datasheet" "https://www.lcsc.com/datasheet/C3681415.pdf"
+			(at 44.45 168.91 0)
+			(hide yes)
+			(show_name no)
+			(do_not_autoplace no)
+			(effects
+				(font
+					(size 1.27 1.27)
+				)
+			)
+		)
+		(property "Description" ""
+			(at 44.45 140.97 0)
+			(hide yes)
+			(show_name no)
+			(do_not_autoplace no)
+			(effects
+				(font
+					(size 1.27 1.27)
+				)
+			)
+		)
+		(property "Manufacturer" "TI(德州仪器)"
+			(at 44.45 171.45 0)
+			(hide yes)
+			(show_name no)
+			(do_not_autoplace no)
+			(effects
+				(font
+					(size 1.27 1.27)
+				)
+			)
+		)
+		(property "MPN" "DRV8328ARUYR"
+			(at 44.45 173.99 0)
+			(hide yes)
+			(show_name no)
+			(do_not_autoplace no)
+			(effects
+				(font
+					(size 1.27 1.27)
+				)
+			)
+		)
+		(property "LCSC Part" "C3681415"
+			(at 44.45 176.53 0)
+			(hide yes)
+			(show_name no)
+			(do_not_autoplace no)
+			(effects
+				(font
+					(size 1.27 1.27)
+				)
+			)
+		)
+		(pin "2"
+		)
+		(pin "4"
+		)
+		(pin "15"
+		)
+		(pin "26"
+		)
+		(pin "28"
+		)
+		(pin "8"
+		)
+		(pin "13"
+		)
+		(pin "27"
+		)
+		(pin "1"
+		)
+		(pin "6"
+		)
+		(pin "5"
+		)
+		(pin "19"
+		)
+		(pin "7"
+		)
+		(pin "3"
+		)
+		(pin "10"
+		)
+		(pin "29"
+		)
+		(pin "22"
+		)
+		(pin "12"
+		)
+		(pin "23"
+		)
+		(pin "21"
+		)
+		(pin "24"
+		)
+		(pin "14"
+		)
+		(pin "25"
+		)
+		(pin "16"
+		)
+		(pin "17"
+		)
+		(pin "18"
+		)
+		(pin "11"
+		)
+		(pin "9"
+		)
+		(pin "20"
+		)
+		(instances
+			(project "espdrone"
+				(path "/d7b09c1f-60ff-44c2-9b85-8e9b4c9b8de4"
+					(reference "U16")
+					(unit 1)
+				)
+			)
+		)
+	)
+	(symbol
 		(lib_name "GND_2")
 		(lib_id "power:GND")
@@
 		(dnp no)
 		(property "Reference" "C28"
-			(at 98.806 78.994 0)
+			(at 98.044 78.994 0)
 			(show_name no)
 			(do_not_autoplace no)
@@
 		)
 		(property "Value" "100u"
-			(at 98.552 81.026 0)
+			(at 97.79 81.026 0)
 			(show_name no)
 			(do_not_autoplace no)
@@
 		(dnp no)
 		(property "Reference" "C26"
-			(at 44.196 78.994 0)
+			(at 43.688 78.994 0)
 			(show_name no)
 			(do_not_autoplace no)
@@
 		)
 		(property "Value" "100u"
-			(at 43.942 81.026 0)
+			(at 43.434 81.026 0)
 			(show_name no)
 			(do_not_autoplace no)
@@
 		(dnp no)
 		(property "Reference" "C24"
-			(at 98.806 35.814 0)
+			(at 98.298 35.814 0)
 			(show_name no)
 			(do_not_autoplace no)
@@
 		)
 		(property "Value" "100u"
-			(at 98.552 37.846 0)
-			(show_name no)
-			(do_not_autoplace no)
+			(at 98.044 37.846 0)
+			(show_name no)
+			(do_not_autoplace no)

Commit message: Restore all functionality from v1
Connections:
- net MOT1 renamed DC_MOT1
- net MOT2 renamed DC_MOT2
- net MOT3 renamed DC_MOT3
- net MOT4 renamed DC_MOT4
Other:
- note added: "Brushed motor drive"
- note removed: "MOTOR DRIVE"
- moved on the sheet: C17, C18, C23, C24, C25, C26, C27, C28, D1, D6, D7, D8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

Commit message: Add beginnings of ESC
Parts:
- removed U16: DRV8328ARUYR, easyeda2kicad:WQFN-28_L4.0-W4.0-P0.40-TL-EP2.6, symbol easyeda2kicad:DRV8328ARUYR
Other:
- moved on the sheet: C17, C18, C23, C24, C25, C26, C27, C28, D1, D6, D7, D8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

Commit message: Improve ESC readability
Other:
- added sheet ESC (esc.kicad_sch)
Changed lines of the file:
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@@
+		)
+	)
+	(sheet
+		(at 175.26 34.29)
+		(size 31.75 40.64)
+		(exclude_from_sim no)
+		(in_bom yes)
+		(on_board yes)
+		(dnp no)
+		(fields_autoplaced yes)
+		(stroke
+			(width 0.1524)
+			(type solid)
+		)
+		(fill
+			(color 0 0 0 0)
+		)
+		(property "Sheetname" "ESC"
+			(at 175.26 33.5784 0)
+			(show_name no)
+			(do_not_autoplace no)
+			(effects
+				(font
+					(size 1.27 1.27)
+				)
+				(justify left bottom)
+			)
+		)
+		(property "Sheetfile" "esc.kicad_sch"
+			(at 175.26 75.5146 0)
+			(show_name no)
+			(do_not_autoplace no)
+			(effects
+				(font
+					(size 1.27 1.27)
+				)
+				(justify left top)
+			)
+		)
+		(instances
+			(project "espdrone"
+				(path "/d7b09c1f-60ff-44c2-9b85-8e9b4c9b8de4"
+					(page "7")
+				)
+			)
 		)
 	)

Commit message: Reorder gate driver symbol and rearrange ESC
Other:
- removed sheet ESC
Changed lines of the file:
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@@
-		)
-	)
-	(sheet
-		(at 175.26 34.29)
-		(size 31.75 40.64)
-		(exclude_from_sim no)
-		(in_bom yes)
-		(on_board yes)
-		(dnp no)
-		(fields_autoplaced yes)
-		(stroke
-			(width 0.1524)
-			(type solid)
-		)
-		(fill
-			(color 0 0 0 0)
-		)
-		(property "Sheetname" "ESC"
-			(at 175.26 33.5784 0)
-			(show_name no)
-			(do_not_autoplace no)
-			(effects
-				(font
-					(size 1.27 1.27)
-				)
-				(justify left bottom)
-			)
-		)
-		(property "Sheetfile" "esc.kicad_sch"
-			(at 175.26 75.5146 0)
-			(show_name no)
-			(do_not_autoplace no)
-			(effects
-				(font
-					(size 1.27 1.27)
-				)
-				(justify left top)
-			)
-		)
-		(instances
-			(project "espdrone"
-				(path "/d7b09c1f-60ff-44c2-9b85-8e9b4c9b8de4"
-					(page "7")
-				)
-			)
 		)
 	)

Commit message: Various little adjustments to ESC
Other:
- added sheet ESC (esc.kicad_sch)
Changed lines of the file:
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@@
+		)
+	)
+	(sheet
+		(at 149.86 20.32)
+		(size 19.05 26.67)
+		(exclude_from_sim no)
+		(in_bom yes)
+		(on_board yes)
+		(dnp no)
+		(fields_autoplaced yes)
+		(stroke
+			(width 0.1524)
+			(type solid)
+		)
+		(fill
+			(color 0 0 0 0)
+		)
+		(property "Sheetname" "ESC"
+			(at 149.86 19.6084 0)
+			(show_name no)
+			(do_not_autoplace no)
+			(effects
+				(font
+					(size 1.27 1.27)
+				)
+				(justify left bottom)
+			)
+		)
+		(property "Sheetfile" "esc.kicad_sch"
+			(at 149.86 47.5746 0)
+			(show_name no)
+			(do_not_autoplace no)
+			(effects
+				(font
+					(size 1.27 1.27)
+				)
+				(justify left top)
+			)
+		)
+		(pin "DSHOT" input
+			(at 149.86 31.75 180)
+			(effects
+				(font
+					(size 1.27 1.27)
+				)
+				(justify left)
+			)
+		)
+		(pin "TELEMETRY" input
+			(at 149.86 35.56 180)
+			(effects
+				(font
+					(size 1.27 1.27)
+				)
+				(justify left)
+			)
+		)
+		(pin "+BATT" input
+			(at 162.56 20.32 90)
+			(effects
+				(font
+					(size 1.27 1.27)
+				)
+				(justify right)
+			)
+		)
+		(pin "3V3" input
+			(at 156.21 20.32 90)
+			(effects
+				(font
+					(size 1.27 1.27)
+				)
+				(justify right)
+			)
+		)
+		(pin "GND" input
+			(at 158.75 46.99 270)
+			(effects
+				(font
+					(size 1.27 1.27)
+				)
+				(justify left)
+			)
+		)
+		(instances
+			(project "espdrone"
+				(path "/d7b09c1f-60ff-44c2-9b85-8e9b4c9b8de4"
+					(page "9")
+				)
+			)
 		)
 	)

Commit message: Move ESCs to motors sheet
Connections:
- no-connect marks 0 -> 4
Other:
- added sheet ESC1 (esc.kicad_sch)
- added sheet ESC2 (esc.kicad_sch)
- added sheet ESC3 (esc.kicad_sch)
- note added: "BLDC motor control"
- note added: "DC motor control"
- note removed: "Brushed motor drive"
