File: motors.kicad_sch (KiCad schematic)
At the start: 32 parts, among them Q1 NMOS, Q2 NMOS, Q3 NMOS, Q4 NMOS

Commit message: Remove a lot of test points
Parts:
- renumbered R57 to R55, R58 to R56, R59 to R57, R60 to R58, R61 to R59, R62 to R60, R63 to R61, R64 to R62
Changed lines of the file:
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@@
 		(in_pos_files yes)
 		(dnp no)
-		(property "Reference" "R63"
+		(property "Reference" "R61"
 			(at 128.524 50.8 0)
 			(show_name no)
@@
 			(project "espdrone"
 				(path "/d7b09c1f-60ff-44c2-9b85-8e9b4c9b8de4"
-					(reference "R63")
+					(reference "R61")
 					(unit 1)
 				)
@@
 		(in_pos_files yes)
 		(dnp no)
-		(property "Reference" "#PWR0164"
+		(property "Reference" "#PWR0163"
 			(at 45.72 80.01 0)
 			(hide yes)
@@
 			(project "espdrone"
 				(path "/d7b09c1f-60ff-44c2-9b85-8e9b4c9b8de4"
-					(reference "#PWR0164")
+					(reference "#PWR0163")
 					(unit 1)
 				)
@@
 		(dnp no)
 		(fields_autoplaced yes)
-		(property "Reference" "#PWR0173"
+		(property "Reference" "#PWR0172"
 			(at 138.43 64.77 0)
 			(hide yes)
@@
 			(project "espdrone"
 				(path "/d7b09c1f-60ff-44c2-9b85-8e9b4c9b8de4"
-					(reference "#PWR0173")
+					(reference "#PWR0172")
 					(unit 1)
 				)
@@
 		(in_pos_files yes)
 		(dnp no)
-		(property "Reference" "R57"
+		(property "Reference" "R55"
 			(at 59.69 50.8 0)
 			(show_name no)
@@
 			(project "espdrone"
 				(path "/d7b09c1f-60ff-44c2-9b85-8e9b4c9b8de4"
-					(reference "R57")
+					(reference "R55")
 					(unit 1)
 				)
@@
 		(dnp no)
 		(fields_autoplaced yes)
-		(property "Reference" "#PWR0174"
+		(property "Reference" "#PWR0173"
 			(at 138.43 111.76 0)
 			(hide yes)
@@
 			(project "espdrone"
 				(path "/d7b09c1f-60ff-44c2-9b85-8e9b4c9b8de4"
-					(reference "#PWR0174")
+					(reference "#PWR0173")
 					(unit 1)
 				)
@@
 		(dnp no)
 		(fields_autoplaced yes)
-		(property "Reference" "#PWR0165"
+		(property "Reference" "#PWR0164"
 			(at 45.72 96.52 0)
 			(hide yes)
@@
 			(project "espdrone"
 				(path "/d7b09c1f-60ff-44c2-9b85-8e9b4c9b8de4"
-					(reference "#PWR0165")
+					(reference "#PWR0164")
 					(unit 1)
 				)
@@
 		(in_pos_files yes)
 		(dnp no)
-		(property "Reference" "R59"
+		(property "Reference" "R57"
 			(at 66.294 50.8 0)
 			(show_name no)
@@
 			(project "espdrone"
 				(path "/d7b09c1f-60ff-44c2-9b85-8e9b4c9b8de4"
-					(reference "R59")
+					(reference "R57")
 					(unit 1)
 				)
@@
 		(in_pos_files yes)
 		(dnp no)
-		(property "Reference" "#PWR0171"
+		(property "Reference" "#PWR0170"
 			(at 107.95 80.01 0)
 			(hide yes)
@@
 			(project "espdrone"
 				(path "/d7b09c1f-60ff-44c2-9b85-8e9b4c9b8de4"
-					(reference "#PWR0171")
+					(reference "#PWR0170")
 					(unit 1)
 				)
@@
 		(dnp no)
 		(fields_autoplaced yes)
-		(property "Reference" "#PWR0167"
+		(property "Reference" "#PWR0166"
 			(at 76.2 111.76 0)
 			(hide yes)
@@
 			(project "espdrone"
 				(path "/d7b09c1f-60ff-44c2-9b85-8e9b4c9b8de4"
-					(reference "#PWR0167")
+					(reference "#PWR0166")
 					(unit 1)
 				)
@@
 		(in_pos_files yes)
 		(dnp no)
-		(property "Reference" "R60"
+		(property "Reference" "R58"
 			(at 63.246 97.79 0)
 			(show_name no)
@@
 			(project "espdrone"
 				(path "/d7b09c1f-60ff-44c2-9b85-8e9b4c9b8de4"
-					(reference "R60")
+					(reference "R58")
 					(unit 1)
 				)
@@
 		(dnp no)
 		(fields_autoplaced yes)
-		(property "Reference" "#PWR0168"
+		(property "Reference" "#PWR0167"
 			(at 97.79 193.04 0)
 			(hide yes)
@@
 			(project "espdrone"
 				(path "/d7b09c1f-60ff-44c2-9b85-8e9b4c9b8de4"
-					(reference "#PWR0168")
+					(reference "#PWR0167")
 					(unit 1)
 				)
@@
 		(in_pos_files yes)
 		(dnp no)
-		(property "Reference" "R61"
+		(property "Reference" "R59"
 			(at 121.92 50.8 0)
 			(show_name no)
@@
 			(project "espdrone"
 				(path "/d7b09c1f-60ff-44c2-9b85-8e9b4c9b8de4"
-					(reference "R61")
+					(reference "R59")
 					(unit 1)
 				)
@@
 		(dnp no)
 		(fields_autoplaced yes)
-		(property "Reference" "#PWR0170"
+		(property "Reference" "#PWR0169"
 			(at 107.95 49.53 0)
 			(hide yes)
@@
 			(project "espdrone"
 				(path "/d7b09c1f-60ff-44c2-9b85-8e9b4c9b8de4"
-					(reference "#PWR0170")
+					(reference "#PWR0169")
 					(unit 1)
 				)
@@
 		(in_pos_files yes)
 		(dnp no)
-		(property "Reference" "#PWR0160"
+		(property "Reference" "#PWR0159"
 			(at 38.1 140.97 0)
 			(hide yes)
@@
 			(project "espdrone"
 				(path "/d7b09c1f-60ff-44c2-9b85-8e9b4c9b8de4"
-					(reference "#PWR0160")
+					(reference "#PWR0159")
 					(unit 1)
 				)
@@
 		(in_pos_files yes)
 		(dnp no)
-		(property "Reference" "R58"
+		(property "Reference" "R56"
 			(at 52.07 97.79 0)
 			(show_name no)
@@
 			(project "espdrone"
 				(path "/d7b09c1f-60ff-44c2-9b85-8e9b4c9b8de4"
-					(reference "R58")
+					(reference "R56")
 					(unit 1)
 				)
@@
 		(dnp no)
 		(fields_autoplaced yes)
-		(property "Reference" "#PWR0163"
+		(property "Reference" "#PWR0162"
 			(at 45.72 49.53 0)
 			(hide yes)
@@
 			(project "espdrone"
 				(path "/d7b09c1f-60ff-44c2-9b85-8e9b4c9b8de4"
-					(reference "#PWR0163")
+					(reference "#PWR0162")
 					(unit 1)
 				)
@@
 		(in_pos_files yes)
 		(dnp no)
-		(property "Reference" "#PWR0169"
+		(property "Reference" "#PWR0168"
 			(at 107.95 33.02 0)
 			(hide yes)
@@
 			(project "espdrone"
 				(path "/d7b09c1f-60ff-44c2-9b85-8e9b4c9b8de4"
-					(reference "#PWR0169")
+					(reference "#PWR0168")
 					(unit 1)
 				)
@@
 		(in_pos_files yes)
 		(dnp no)
-		(property "Reference" "#PWR0161"
+		(property "Reference" "#PWR0160"
 			(at 44.45 140.97 0)
 			(hide yes)
@@
 			(project "espdrone"
 				(path "/d7b09c1f-60ff-44c2-9b85-8e9b4c9b8de4"
-					(reference "#PWR0161")
+					(reference "#PWR0160")
 					(unit 1)
 				)
@@
 		(dnp no)
 		(fields_autoplaced yes)
-		(property "Reference" "#PWR0172"
+		(property "Reference" "#PWR0171"
 			(at 107.95 96.52 0)
 			(hide yes)
@@
 			(project "espdrone"
 				(path "/d7b09c1f-60ff-44c2-9b85-8e9b4c9b8de4"
-					(reference "#PWR0172")
+					(reference "#PWR0171")
 					(unit 1)
 				)
@@
 		(in_pos_files yes)
 		(dnp no)
-		(property "Reference" "R64"
+		(property "Reference" "R62"
 			(at 128.524 97.79 0)
 			(show_name no)
@@
 			(project "espdrone"
 				(path "/d7b09c1f-60ff-44c2-9b85-8e9b4c9b8de4"
-					(reference "R64")
+					(reference "R62")
 					(unit 1)
 				)
@@
 		(dnp no)
 		(fields_autoplaced yes)
-		(property "Reference" "#PWR0166"
+		(property "Reference" "#PWR0165"
 			(at 76.2 64.77 0)
 			(hide yes)
@@
 			(project "espdrone"
 				(path "/d7b09c1f-60ff-44c2-9b85-8e9b4c9b8de4"
-					(reference "#PWR0166")
+					(reference "#PWR0165")
 					(unit 1)
 				)
@@
 		(in_pos_files yes)
 		(dnp no)
-		(property "Reference" "#PWR0162"
+		(property "Reference" "#PWR0161"
 			(at 45.72 33.02 0)
 			(hide yes)
@@
 			(project "espdrone"
 				(path "/d7b09c1f-60ff-44c2-9b85-8e9b4c9b8de4"
-					(reference "#PWR0162")
+					(reference "#PWR0161")
 					(unit 1)
 				)
@@
 		(in_pos_files yes)
 		(dnp no)
-		(property "Reference" "R62"
+		(property "Reference" "R60"
 			(at 121.92 97.79 0)
 			(show_name no)
@@
 			(project "espdrone"
 				(path "/d7b09c1f-60ff-44c2-9b85-8e9b4c9b8de4"
-					(reference "R62")
+					(reference "R60")
 					(unit 1)
 				)

Commit message: Remove whole battery current shunt and replace MOSFETs with 3.3x3.3mm alternative
Parts:
- C100, C101, C96, C97: footprint Capacitor_SMD:C_0603_1608Metric -> Capacitor_SMD:C_0402_1005Metric
- R55, R56, R57, R58, R59, R60, R61, R62: footprint Resistor_SMD:R_0603_1608Metric -> Resistor_SMD:R_0402_1005Metric
- TP10, TP3, TP4, TP5, TP6, TP7, TP8, TP9: footprint TestPoint:TestPoint_Pad_2.0x2.0mm -> TestPoint:TestPoint_Pad_1.5x1.5mm
Changed lines of the file:
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@@
 			)
 		)
-		(property "Footprint" "Resistor_SMD:R_0603_1608Metric"
+		(property "Footprint" "Resistor_SMD:R_0402_1005Metric"
 			(at 125.222 52.07 90)
 			(hide yes)
@@
 			)
 		)
-		(property "Footprint" "Resistor_SMD:R_0603_1608Metric"
+		(property "Footprint" "Resistor_SMD:R_0402_1005Metric"
 			(at 57.658 52.07 90)
 			(hide yes)
@@
 			)
 		)
-		(property "Footprint" "TestPoint:TestPoint_Pad_2.0x2.0mm"
+		(property "Footprint" "TestPoint:TestPoint_Pad_1.5x1.5mm"
 			(at 128.27 30.48 0)
 			(hide yes)
@@
 			)
 		)
-		(property "Footprint" "TestPoint:TestPoint_Pad_2.0x2.0mm"
+		(property "Footprint" "TestPoint:TestPoint_Pad_1.5x1.5mm"
 			(at 128.27 77.47 0)
 			(hide yes)
@@
 			)
 		)
-		(property "Footprint" "Capacitor_SMD:C_0603_1608Metric"
+		(property "Footprint" "Capacitor_SMD:C_0402_1005Metric"
 			(at 44.7548 40.64 0)
 			(hide yes)
@@
 			)
 		)
-		(property "Footprint" "Resistor_SMD:R_0603_1608Metric"
+		(property "Footprint" "Resistor_SMD:R_0402_1005Metric"
 			(at 62.992 52.07 90)
 			(hide yes)
@@
 			)
 		)
-		(property "Footprint" "TestPoint:TestPoint_Pad_2.0x2.0mm"
+		(property "Footprint" "TestPoint:TestPoint_Pad_1.5x1.5mm"
 			(at 143.51 30.48 0)
 			(hide yes)
@@
 			)
 		)
-		(property "Footprint" "TestPoint:TestPoint_Pad_2.0x2.0mm"
+		(property "Footprint" "TestPoint:TestPoint_Pad_1.5x1.5mm"
 			(at 66.04 30.48 0)
 			(hide yes)
@@
 			)
 		)
-		(property "Footprint" "TestPoint:TestPoint_Pad_2.0x2.0mm"
+		(property "Footprint" "TestPoint:TestPoint_Pad_1.5x1.5mm"
 			(at 66.04 77.47 0)
 			(hide yes)
@@
 			)
 		)
-		(property "Footprint" "Resistor_SMD:R_0603_1608Metric"
+		(property "Footprint" "Resistor_SMD:R_0402_1005Metric"
 			(at 66.548 99.06 90)
 			(hide yes)
@@
 			)
 		)
-		(property "Footprint" "TestPoint:TestPoint_Pad_2.0x2.0mm"
+		(property "Footprint" "TestPoint:TestPoint_Pad_1.5x1.5mm"
 			(at 143.51 77.47 0)
 			(hide yes)
@@
 			)
 		)
-		(property "Footprint" "Resistor_SMD:R_0603_1608Metric"
+		(property "Footprint" "Resistor_SMD:R_0402_1005Metric"
 			(at 119.888 52.07 90)
 			(hide yes)
@@
 			)
 		)
-		(property "Footprint" "TestPoint:TestPoint_Pad_2.0x2.0mm"
+		(property "Footprint" "TestPoint:TestPoint_Pad_1.5x1.5mm"
 			(at 81.28 77.47 0)
 			(hide yes)
@@
 			)
 		)
-		(property "Footprint" "Capacitor_SMD:C_0603_1608Metric"
+		(property "Footprint" "Capacitor_SMD:C_0402_1005Metric"
 			(at 44.7548 87.63 0)
 			(hide yes)
@@
 			)
 		)
-		(property "Footprint" "Resistor_SMD:R_0603_1608Metric"
+		(property "Footprint" "Resistor_SMD:R_0402_1005Metric"
 			(at 54.102 99.06 90)
 			(hide yes)
@@
 			)
 		)
-		(property "Footprint" "Capacitor_SMD:C_0603_1608Metric"
+		(property "Footprint" "Capacitor_SMD:C_0402_1005Metric"
 			(at 106.9848 87.63 0)
 			(hide yes)
@@
 			)
 		)
-		(property "Footprint" "Resistor_SMD:R_0603_1608Metric"
+		(property "Footprint" "Resistor_SMD:R_0402_1005Metric"
 			(at 125.222 99.06 90)
 			(hide yes)
@@
 			)
 		)
-		(property "Footprint" "TestPoint:TestPoint_Pad_2.0x2.0mm"
+		(property "Footprint" "TestPoint:TestPoint_Pad_1.5x1.5mm"
 			(at 81.28 30.48 0)
 			(hide yes)
@@
 			)
 		)
-		(property "Footprint" "Capacitor_SMD:C_0603_1608Metric"
+		(property "Footprint" "Capacitor_SMD:C_0402_1005Metric"
 			(at 106.9848 40.64 0)
 			(hide yes)
@@
 			)
 		)
-		(property "Footprint" "Resistor_SMD:R_0603_1608Metric"
+		(property "Footprint" "Resistor_SMD:R_0402_1005Metric"
 			(at 119.888 99.06 90)
 			(hide yes)

Commit message: Improve some connector footprints
Parts:
- TP10, TP3, TP4, TP5, TP6, TP7, TP8, TP9: footprint TestPoint:TestPoint_Pad_1.5x1.5mm -> easyeda2kicad:MotorPad_1x3mm
- renumbered C102 to C100, C103 to C101, C96 to C94, C97 to C95, C98 to C96, C99 to C97, C100 to C98, C101 to C99, R55 to R53, R56 to R54, R57 to R55, R58 to R56, R59 to R57, R60 to R58, R61 to R59, R62 to R60
Other:
- removed sheet ESC
- added sheet ESC4 (esc.kicad_sch)
Changed lines of the file:
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@@
 		(in_pos_files yes)
 		(dnp no)
-		(property "Reference" "R61"
+		(property "Reference" "R59"
 			(at 128.524 50.8 0)
 			(show_name no)
@@
 			(project "espdrone"
 				(path "/d7b09c1f-60ff-44c2-9b85-8e9b4c9b8de4"
-					(reference "R61")
+					(reference "R59")
 					(unit 1)
 				)
@@
 		(in_pos_files yes)
 		(dnp no)
-		(property "Reference" "C98"
+		(property "Reference" "C96"
 			(at 50.038 35.814 0)
 			(show_name no)
@@
 			(project "espdrone"
 				(path "/d7b09c1f-60ff-44c2-9b85-8e9b4c9b8de4"
-					(reference "C98")
+					(reference "C96")
 					(unit 1)
 				)
@@
 		(in_pos_files yes)
 		(dnp no)
-		(property "Reference" "R55"
+		(property "Reference" "R53"
 			(at 59.69 50.8 0)
 			(show_name no)
@@
 			(project "espdrone"
 				(path "/d7b09c1f-60ff-44c2-9b85-8e9b4c9b8de4"
-					(reference "R55")
+					(reference "R53")
 					(unit 1)
 				)
@@
 			)
 		)
-		(property "Footprint" "TestPoint:TestPoint_Pad_1.5x1.5mm"
+		(property "Footprint" "easyeda2kicad:MotorPad_1x3mm"
 			(at 128.27 30.48 0)
 			(hide yes)
@@
 			)
 		)
-		(property "Footprint" "TestPoint:TestPoint_Pad_1.5x1.5mm"
+		(property "Footprint" "easyeda2kicad:MotorPad_1x3mm"
 			(at 128.27 77.47 0)
 			(hide yes)
@@
 		(in_pos_files yes)
 		(dnp no)
-		(property "Reference" "C96"
+		(property "Reference" "C94"
 			(at 41.91 35.5599 0)
 			(show_name no)
@@
 			(project "espdrone"
 				(path "/d7b09c1f-60ff-44c2-9b85-8e9b4c9b8de4"
-					(reference "C96")
+					(reference "C94")
 					(unit 1)
 				)
@@
 		(in_pos_files yes)
 		(dnp no)
-		(property "Reference" "R57"
+		(property "Reference" "R55"
 			(at 66.294 50.8 0)
 			(show_name no)
@@
 			(project "espdrone"
 				(path "/d7b09c1f-60ff-44c2-9b85-8e9b4c9b8de4"
-					(reference "R57")
+					(reference "R55")
 					(unit 1)
 				)
@@
 			)
 		)
-		(property "Footprint" "TestPoint:TestPoint_Pad_1.5x1.5mm"
+		(property "Footprint" "easyeda2kicad:MotorPad_1x3mm"
 			(at 143.51 30.48 0)
 			(hide yes)
@@
 			)
 		)
-		(property "Footprint" "TestPoint:TestPoint_Pad_1.5x1.5mm"
+		(property "Footprint" "easyeda2kicad:MotorPad_1x3mm"
 			(at 66.04 30.48 0)
 			(hide yes)
@@
 			)
 		)
-		(property "Footprint" "TestPoint:TestPoint_Pad_1.5x1.5mm"
+		(property "Footprint" "easyeda2kicad:MotorPad_1x3mm"
 			(at 66.04 77.47 0)
 			(hide yes)
@@
 		(in_pos_files yes)
 		(dnp no)
-		(property "Reference" "R58"
+		(property "Reference" "R56"
 			(at 63.246 97.79 0)
 			(show_name no)
@@
 			(project "espdrone"
 				(path "/d7b09c1f-60ff-44c2-9b85-8e9b4c9b8de4"
-					(reference "R58")
+					(reference "R56")
 					(unit 1)
 				)
@@
 		(in_pos_files yes)
 		(dnp no)
-		(property "Reference" "C103"
+		(property "Reference" "C101"
 			(at 112.014 82.804 0)
 			(show_name no)
@@
 			(project "espdrone"
 				(path "/d7b09c1f-60ff-44c2-9b85-8e9b4c9b8de4"
-					(reference "C103")
+					(reference "C101")
 					(unit 1)
 				)
@@
 		(in_pos_files yes)
 		(dnp no)
-		(property "Reference" "C99"
+		(property "Reference" "C97"
 			(at 50.038 82.804 0)
 			(show_name no)
@@
 			(project "espdrone"
 				(path "/d7b09c1f-60ff-44c2-9b85-8e9b4c9b8de4"
-					(reference "C99")
+					(reference "C97")
 					(unit 1)
 				)
@@
 			)
 		)
-		(property "Footprint" "TestPoint:TestPoint_Pad_1.5x1.5mm"
+		(property "Footprint" "easyeda2kicad:MotorPad_1x3mm"
 			(at 143.51 77.47 0)
 			(hide yes)
@@
 		(in_pos_files yes)
 		(dnp no)
-		(property "Reference" "R59"
+		(property "Reference" "R57"
 			(at 121.92 50.8 0)
 			(show_name no)
@@
 			(project "espdrone"
 				(path "/d7b09c1f-60ff-44c2-9b85-8e9b4c9b8de4"
-					(reference "R59")
+					(reference "R57")
 					(unit 1)
 				)
@@
 			)
 		)
-		(property "Footprint" "TestPoint:TestPoint_Pad_1.5x1.5mm"
+		(property "Footprint" "easyeda2kicad:MotorPad_1x3mm"
 			(at 81.28 77.47 0)
 			(hide yes)
@@
 		(in_pos_files yes)
 		(dnp no)
-		(property "Reference" "C97"
+		(property "Reference" "C95"
 			(at 41.91 82.5499 0)
 			(show_name no)
@@
 			(project "espdrone"
 				(path "/d7b09c1f-60ff-44c2-9b85-8e9b4c9b8de4"
-					(reference "C97")
+					(reference "C95")
 					(unit 1)
 				)
@@
 		(in_pos_files yes)
 		(dnp no)
-		(property "Reference" "R56"
+		(property "Reference" "R54"
 			(at 52.07 97.79 0)
 			(show_name no)
@@
 			(project "espdrone"
 				(path "/d7b09c1f-60ff-44c2-9b85-8e9b4c9b8de4"
-					(reference "R56")
+					(reference "R54")
 					(unit 1)
 				)
@@
 		(in_pos_files yes)
 		(dnp no)
-		(property "Reference" "C101"
+		(property "Reference" "C99"
 			(at 104.14 82.5499 0)
 			(show_name no)
@@
 			(project "espdrone"
 				(path "/d7b09c1f-60ff-44c2-9b85-8e9b4c9b8de4"
-					(reference "C101")
+					(reference "C99")
 					(unit 1)
 				)
@@
 		(in_pos_files yes)
 		(dnp no)
-		(property "Reference" "C102"
+		(property "Reference" "C100"
 			(at 112.268 35.814 0)
 			(show_name no)
@@
 			(project "espdrone"
 				(path "/d7b09c1f-60ff-44c2-9b85-8e9b4c9b8de4"
-					(reference "C102")
+					(reference "C100")
 					(unit 1)
 				)
@@
 		(in_pos_files yes)
 		(dnp no)
-		(property "Reference" "R62"
+		(property "Reference" "R60"
 			(at 128.524 97.79 0)
 			(show_name no)
@@
 			(project "espdrone"
 				(path "/d7b09c1f-60ff-44c2-9b85-8e9b4c9b8de4"
-					(reference "R62")
+					(reference "R60")
 					(unit 1)
 				)
@@
 			)
 		)
-		(property "Footprint" "TestPoint:TestPoint_Pad_1.5x1.5mm"
+		(property "Footprint" "easyeda2kicad:MotorPad_1x3mm"
 			(at 81.28 30.48 0)
 			(hide yes)
@@
 		(in_pos_files yes)
 		(dnp no)
-		(property "Reference" "C100"
+		(property "Reference" "C98"
 			(at 104.14 35.5599 0)
 			(show_name no)
@@
 			(project "espdrone"
 				(path "/d7b09c1f-60ff-44c2-9b85-8e9b4c9b8de4"
-					(reference "C100")
+					(reference "C98")
 					(unit 1)
 				)
@@
 		(in_pos_files yes)
 		(dnp no)
-		(property "Reference" "R60"
+		(property "Reference" "R58"
 			(at 121.92 97.79 0)
 			(show_name no)
@@
 			(project "espdrone"
 				(path "/d7b09c1f-60ff-44c2-9b85-8e9b4c9b8de4"
-					(reference "R60")
+					(reference "R58")
 					(unit 1)
 				)
@@
 			(color 0 0 0 0)
 		)
-		(property "Sheetname" "ESC1"
+		(property "Sheetname" "ESC2"
 			(at 69.85 151.6884 0)
 			(show_name no)
@@
 			(color 0 0 0 0)
 		)
-		(property "Sheetname" "ESC3"
+		(property "Sheetname" "ESC4"
 			(at 146.05 151.6884 0)
 			(show_name no)
@@
 			(color 0 0 0 0)
 		)
-		(property "Sheetname" "ESC2"
+		(property "Sheetname" "ESC3"
 			(at 107.95 151.6884 0)
 			(show_name no)
@@
 			(color 0 0 0 0)
 		)
-		(property "Sheetname" "ESC"
+		(property "Sheetname" "ESC1"
 			(at 31.75 151.6884 0)
 			(show_name no)

Commit message: Ostensibly finish ESC routing
Connections:
- no-connect marks 4 -> 0
Changed lines of the file:
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@@
 		(color 0 0 0 0)
 	)
-	(no_connect
-		(at 107.95 167.64)
-	)
-	(no_connect
-		(at 146.05 167.64)
-	)
-	(no_connect
-		(at 69.85 167.64)
-	)
-	(no_connect
-		(at 31.75 167.64)
-	)
 	(wire
 		(pts
@@
 	(wire
 		(pts
+			(xy 67.31 167.64) (xy 69.85 167.64)
+		)
+		(stroke
+			(width 0)
+			(type default)
+		)
+	)
+	(wire
+		(pts
 			(xy 76.2 52.07) (xy 76.2 57.15)
 		)
@@
 	(wire
 		(pts
+			(xy 29.21 167.64) (xy 31.75 167.64)
+		)
+		(stroke
+			(width 0)
+			(type default)
+		)
+	)
+	(wire
+		(pts
 			(xy 55.88 55.88) (xy 55.88 57.15)
 		)
@@
 	(wire
 		(pts
+			(xy 143.51 167.64) (xy 146.05 167.64)
+		)
+		(stroke
+			(width 0)
+			(type default)
+		)
+	)
+	(wire
+		(pts
 			(xy 64.77 46.99) (xy 68.58 46.99)
 		)
@@
 		(pts
 			(xy 55.88 93.98) (xy 64.77 93.98)
+		)
+		(stroke
+			(width 0)
+			(type default)
+		)
+	)
+	(wire
+		(pts
+			(xy 105.41 167.64) (xy 107.95 167.64)
 		)
 		(stroke
@@
 		)
 	)
+	(global_label "TELEMETRY"
+		(shape input)
+		(at 67.31 167.64 180)
+		(fields_autoplaced yes)
+		(effects
+			(font
+				(size 1.27 1.27)
+			)
+			(justify right)
+		)
+		(property "Intersheetrefs" "${INTERSHEET_REFS}"
+			(at 54.1045 167.64 0)
+			(hide yes)
+			(show_name no)
+			(do_not_autoplace no)
+			(effects
+				(font
+					(size 1.27 1.27)
+				)
+				(justify right)
+			)
+		)
+	)
 	(global_label "DC_MOT1"
 		(shape input)
@@
 		)
 	)
+	(global_label "TELEMETRY"
+		(shape input)
+		(at 143.51 167.64 180)
+		(fields_autoplaced yes)
+		(effects
+			(font
+				(size 1.27 1.27)
+			)
+			(justify right)
+		)
+		(property "Intersheetrefs" "${INTERSHEET_REFS}"
+			(at 130.3045 167.64 0)
+			(hide yes)
+			(show_name no)
+			(do_not_autoplace no)
+			(effects
+				(font
+					(size 1.27 1.27)
+				)
+				(justify right)
+			)
+		)
+	)
 	(global_label "DC_MOT4"
 		(shape input)
@@
 			(hide yes)
 			(show_name no)
+			(do_not_autoplace no)
+			(effects
+				(font
+					(size 1.27 1.27)
+				)
+				(justify right)
+			)
+		)
+	)
+	(global_label "TELEMETRY"
+		(shape input)
+		(at 105.41 167.64 180)
+		(fields_autoplaced yes)
+		(effects
+			(font
+				(size 1.27 1.27)
+			)
+			(justify right)
+		)
+		(property "Intersheetrefs" "${INTERSHEET_REFS}"
+			(at 92.2045 167.64 0)
+			(hide yes)
+			(show_name no)
+			(do_not_autoplace no)
+			(effects
+				(font
+					(size 1.27 1.27)
+				)
+				(justify right)
+			)
+		)
+	)
+	(global_label "TELEMETRY"
+		(shape input)
+		(at 29.21 167.64 180)
+		(fields_autoplaced yes)
+		(effects
+			(font
+				(size 1.27 1.27)
+			)
+			(justify right)
+		)
+		(property "Intersheetrefs" "${INTERSHEET_REFS}"
+			(at 16.0045 167.64 0)
+			(hide yes)
+			(show_name no)

Commit message: Fix DC motor MOSFET footprint
Parts:
- Q1, Q2, Q3, Q4: footprint Package_TO_SOT_SMD:SOT-23 -> easyeda2kicad:SOT-23-IRLML6344
Changed lines of the file:
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@@
 			)
 		)
-		(property "Footprint" "Package_TO_SOT_SMD:SOT-23"
+		(property "Footprint" "easyeda2kicad:SOT-23-IRLML6344"
 			(at 78.74 44.45 0)
 			(hide yes)
@@
 			)
 		)
-		(property "Footprint" "Package_TO_SOT_SMD:SOT-23"
+		(property "Footprint" "easyeda2kicad:SOT-23-IRLML6344"
 			(at 140.97 91.44 0)
 			(hide yes)
@@
 			)
 		)
-		(property "Footprint" "Package_TO_SOT_SMD:SOT-23"
+		(property "Footprint" "easyeda2kicad:SOT-23-IRLML6344"
 			(at 140.97 44.45 0)
 			(hide yes)
@@
 			)
 		)
-		(property "Footprint" "Package_TO_SOT_SMD:SOT-23"
+		(property "Footprint" "easyeda2kicad:SOT-23-IRLML6344"
 			(at 78.74 91.44 0)
 			(hide yes)
